File: hot65.kicad_pcb (KiCad board)
At the start: 2 copper layers, 285 x 95 mm, 152 parts, among them P1 USB_C_Plug_USB2.0, SW1 SW_Push, SW10 SW_Push, SW11 SW_Push, SW12 SW_Push, SW13 SW_Push, SW14 SW_Push, SW15 SW_Push, SW16 SW_Push, SW17 SW_Push, SW18 SW_Push, SW19 SW_Push, SW2 SW_Push, SW20 SW_Push, SW21 SW_Push, SW22 SW_Push, SW23 SW_Push, SW24 SW_Push, SW25 SW_Push, SW26 SW_Push, SW27 SW_Push, SW28 SW_Push, SW29 SW_Push, SW3 SW_Push, SW30 SW_Push, SW31 SW_Push, SW32 SW_Push, SW33 SW_Push, SW34 SW_Push, SW35 SW_Push, SW36 SW_Push, SW37 SW_Push, SW38 SW_Push, SW39 SW_Push, SW4 SW_Push, SW40 SW_Push, SW41 SW_Push, SW42 SW_Push, SW43 SW_Push, SW44 SW_Push, SW45 SW_Push, SW46 SW_Push, SW47 SW_Push, SW48 SW_Push, SW49 SW_Push, SW5 SW_Push, SW50 SW_Push, SW51 SW_Push, SW52 SW_Push, SW53 SW_Push, SW54 SW_Push, SW55 SW_Push, SW56 SW_Push, SW57 SW_Push, SW58 SW_Push, SW59 SW_Push, SW6 SW_Push, SW60 SW_Push, SW61 SW_Push, SW62 SW_Push, SW63 SW_Push, SW64 SW_Push, SW65 SW_Push, SW7 SW_Push, SW8 SW_Push, SW9 SW_Push, U1 ATmega32U4-AU, Y1 Crystal_Small

Commit message: v.0.7
Parts:
- added D65: D_Small, Diode_THT:D_T-1_P5.08mm_Horizontal, B.Cu at (84.4, 83.8)
- added D66: D_Small, Diode_THT:D_T-1_P5.08mm_Horizontal, B.Cu at (115.3, 83.8)
- added D67: D_Small, Diode_THT:D_T-1_P5.08mm_Horizontal, B.Cu at (155.6, 83.8)
- added J1: Debug, Connector_PinHeader_1.00mm:PinHeader_1x06_P1.00mm_Vertical, B.Cu at (17.5, 19.1)
- added SW66: SW_Push, MXSocketAlps:MXSocketAlps_2u, F.Cu at (80.8, 76.0)
- added SW67: SW_Push, MXSocketAlps:MXSocketAlps_1.25u, F.Cu at (111.6, 76.0)
- added SW68: SW_Push, MXSocketAlps:MXSocketAlps_3u, F.Cu at (152.0, 76.0)
- D1, D10, D11, D12, D13, D14, D15, D16, D17, D18, D19, D2, D20, D21, D22, D23, D24, D25, D26, D27, D28, D29, D3, D30, D31, D32, D33, D34, D35, D36, D37, D38, D39, D4, D40, D41, D42, D43, D44, D45, D46, D47, D48, D49, D5, D50, D51, D52, D53, D54, D55, D56, D57, D58, D59, D6, D60, D61, D62, D63, D64, D7, D8, D9: footprint Diode_THT:D_A-405_P5.08mm_Vertical_AnodeUp -> Diode_THT:D_T-1_P5.08mm_Horizontal
- H1, H2, H3, H4, H5, H6: moved to B.Cu
- SW10, SW12, SW13, SW14, SW15, SW17, SW18, SW19, SW2, SW20, SW21, SW22, SW23, SW24, SW25, SW26, SW27, SW28, SW30, SW31, SW32, SW33, SW34, SW35, SW36, SW37, SW38, SW39, SW40, SW41, SW42, SW43, SW44, SW45, SW46, SW47, SW48, SW49, SW50, SW51, SW52, SW53, SW54, SW55, SW56, SW57, SW58, SW59, SW60, SW64, SW65, SW7, SW8, SW9: footprint keyswitches:Socket MX Alps -> MXSocketAlps:MXSocketAlps
- SW11, SW16, SW6: footprint keyswitches:Socket MX Alps -> MXSocketAlps:MXSocketAlps_1.25u
- SW29: footprint keyboardstuff:MXSocketAlps_6.25u -> MXSocketAlps:MXSocketAlps_6.25u
- SW3, SW62: footprint keyswitches:Socket MX Alps -> MXSocketAlps:MXSocketAlps_1.5u
- SW4: footprint keyswitches:Socket MX Alps -> MXSocketAlps:MXSocketAlps _1.75u
- SW5, SW61: footprint keyboardstuff:MXSocketAlps_2u -> MXSocketAlps:MXSocketAlps_2u
- SW63: footprint keyboardstuff:MXSocketAlps_2.25u -> MXSocketAlps:MXSocketAlps_2.25u
- moved R6 324.8 mm to (-5.69, -31.4)
- moved C8 318.0 mm to (-5.69, -16.4)
- moved D1 296.1 mm to (2.60, 9.50), turned to 180 degrees
- moved D6 288.0 mm to (21.6, 9.50), turned to 180 degrees
- moved D2 285.0 mm to (7.20, 28.5), turned to 180 degrees
- moved D7 284.0 mm to (20.8, 21.4), turned to 90 degrees
- moved D4 283.3 mm to (12.0, 66.5), turned to 180 degrees
- moved C2 283.0 mm to (39.3, -28.2)
- moved C5 282.3 mm to (39.3, -23.2)
- moved D10 279.8 mm to (29.8, 83.8), turned to 180 degrees
- moved C1 279.7 mm to (39.3, -18.2)
- moved R5 279.6 mm to (27.3, 27.4)
- moved C4 278.1 mm to (39.3, -25.7)
- moved C7 276.7 mm to (30.6, 27.4)
- moved C6 274.0 mm to (33.9, 27.4)
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Connections:
- net Net-(R5-Pad2) renamed RESET
- U1 pad 10: Net-(U1-Pad10) -> MOSI
- U1 pad 11: Net-(U1-Pad11) -> MISO
- U1 pad 9: Net-(U1-Pad9) -> SCLK
Routing:
- net row4: track 0.00 -> 275.9 mm
- net col4: track 0.00 -> 53.1 mm
- net col0: track 0.00 -> 48.6 mm, vias 0 -> 1
- net col13: track 0.00 -> 47.1 mm
- net col3: track 0.00 -> 47.1 mm
- net col1: track 0.00 -> 47.1 mm
- net col2: track 0.00 -> 47.1 mm
- net col6: track 0.00 -> 47.1 mm
- net col9: track 0.00 -> 47.1 mm
- net col11: track 0.00 -> 47.1 mm
- net col10: track 0.00 -> 47.1 mm
- net col5: track 0.00 -> 37.7 mm
- net col12: track 0.00 -> 37.7 mm
- net col8: track 0.00 -> 37.7 mm
- net col7: track 0.00 -> 37.7 mm
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- added copper zone on B.Cu, net GND
- added copper zone on F.Cu, net GND
Other:
- outline, holes or cut-outs redrawn

Commit message: v.1.0
Parts:
- removed P1: USB_C_Plug_USB2.0, Connector_USB:USB_C_Receptacle_HRO_TYPE-C-31-M-12
- added D68: LED_Small, LED_SMD:LED_0603_1608Metric, B.Cu at (7.81, 8.62)
- added J2: USB_C_Receptacle_USB2.0, Connector_USB:USB_C_Receptacle_XKB_U262-16XN-4BVC11, B.Cu at (9.05, -7.37)
- added R7: 22, Resistor_SMD:R_0603_1608Metric_Pad0.98x0.95mm_HandSolder, B.Cu at (7.92, 10.4)
- added U2: USBLC6-2SC6, Package_TO_SOT_SMD:SOT-23-6, B.Cu at (9.60, -0.72)
- H1, H2, H3, H4: footprint MountingHole:MountingHole_2.2mm_M2_DIN965 -> keyboardstuff:M2_slot; moved to F.Cu
- H5, H6: footprint MountingHole:MountingHole_2.2mm_M2_DIN965 -> keyboardstuff:M2_long_slot; moved to F.Cu
- J1: value Debug -> Conn_02x03_Top_Bottom; footprint Connector_PinHeader_1.00mm:PinHeader_1x06_P1.00mm_Vertical -> Connector_PinHeader_1.00mm:PinHeader_2x03_P1.00mm_Vertical
- SW4: footprint MXSocketAlps:MXSocketAlps _1.75u -> MXSocketAlps:MXSocketAlps_1.75u
- moved H5 269.0 mm to (275.9, 47.3)
- moved H6 266.3 mm to (-9.15, 47.3)
- moved H3 153.1 mm to (181.3, 76.0)
- moved H1 79.6 mm to (16.1, 18.7)
- moved R6 79.0 mm to (20.9, 43.0), turned to 90 degrees
- moved C2 68.6 mm to (26.5, 39.1), turned to 90 degrees
- moved C5 60.5 mm to (11.8, 30.7), turned to 315 degrees
- moved C3 59.9 mm to (19.6, 43.0), turned to 90 degrees
- moved C4 57.8 mm to (15.5, 26.9), turned to 315 degrees
- moved H2 52.8 mm to (119.0, 37.8)
- moved C8 48.7 mm to (14.5, 27.9), turned to 135 degrees
- moved C1 47.3 mm to (24.7, 26.8), turned to 180 degrees
- moved R4 39.9 mm to (11.6, 9.55), turned to 90 degrees
- moved R3 37.1 mm to (10.2, 9.55), turned to 270 degrees
- moved H4 16.3 mm to (250.9, 18.7)
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Connections:
- J1 pad 1: RESET -> MISO
- J1 pad 2: MISO -> SCLK
- J1 pad 3: MOSI -> RESET
- J1 pad 4: SCLK -> VCC
- J1 pad 5: GND -> MOSI
- J1 pad 6: VCC -> GND
- R1 pad 1: VCC -> GND
- R2 pad 2: VCC -> GND
- R4 pad 1: Net-(P1-PadA6) -> D+
- R4 pad 2: D+ -> Net-(R4-Pad2)
- U1 pad 18: Net-(U1-Pad18) -> col13
- U1 pad 19: Net-(U1-Pad19) -> col12
- U1 pad 20: Net-(U1-Pad20) -> col11
- U1 pad 21: Net-(U1-Pad21) -> col10
- U1 pad 22: Net-(U1-Pad22) -> col9
- U1 pad 25: Net-(U1-Pad25) -> col8
- U1 pad 26: Net-(U1-Pad26) -> col7
- U1 pad 27: Net-(U1-Pad27) -> col6
- U1 pad 28: Net-(U1-Pad28) -> col5
- U1 pad 29: Net-(U1-Pad29) -> col4
- U1 pad 30: Net-(U1-Pad30) -> col3
- U1 pad 31: Net-(U1-Pad31) -> col2
- U1 pad 32: Net-(U1-Pad32) -> col1
- U1 pad 36: Net-(U1-Pad36) -> row4
- U1 pad 37: Net-(U1-Pad37) -> row3
- U1 pad 38: Net-(U1-Pad38) -> col0
- U1 pad 39: Net-(U1-Pad39) -> row0
- U1 pad 40: Net-(U1-Pad40) -> row2
- U1 pad 41: Net-(U1-Pad41) -> row1
Routing:
- net row0: track 0.00 -> 444.5 mm
- net row1: track 0.00 -> 340.4 mm
- net row3: track 0.00 -> 337.3 mm
- net row2: track 0.00 -> 327.4 mm, vias 0 -> 1
- net col13: track 47.1 -> 344.9 mm, vias 0 -> 4
- net col12: track 37.7 -> 326.2 mm, vias 0 -> 2
- net col11: track 47.1 -> 303.9 mm, vias 0 -> 2
- net col10: track 47.1 -> 284.1 mm, vias 0 -> 2
- net col9: track 47.1 -> 264.4 mm, vias 0 -> 2
- net col8: track 37.7 -> 240.8 mm, vias 0 -> 4
- net col7: track 37.7 -> 221.5 mm, vias 0 -> 4
- net col6: track 47.1 -> 228.8 mm, vias 0 -> 2
- net col5: track 37.7 -> 203.2 mm, vias 0 -> 2
- net col4: track 53.1 -> 195.0 mm, vias 0 -> 2
- net col3: track 47.1 -> 164.5 mm, vias 0 -> 2
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Other:
- board size 285 x 95 mm -> 285 x 94.6 mm

Commit message: v.1.1 Fixed drill errors
Other:
- net class Default: clearance 0.2 -> 0.127
- rule trace_clearance: 0.2 -> 0.127
